File: hardware/Design-1-Draft.kicad_sch (KiCad schematic)
At the start: 32 parts, among them J1 Barrel_Jack_Switch, M1 WATERPUMP-1, M2 WATERPUMP-2, Q1 IRLZ44N, Q2 IRLZ44N, SW1 Button, U3 ADS1115IDGS, U5 Tang_Nano_9K

Commit message: some updates footprint and pcb
Parts:
- BZ1, SW1: footprint (none) -> Connector_PinHeader_2.54mm:PinHeader_1x02_P2.54mm_Vertical
- F1: footprint (none) -> Fuse:Fuseholder_Clip-5x20mm_Keystone_3512P_Inline_P23.62x7.27mm_D1.02x2.41x1.02x1.57mm_Horizontal
Changed lines of the file:
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@@
 			)
 		)
-		(property "Footprint" ""
+		(property "Footprint" "Fuse:Fuseholder_Clip-5x20mm_Keystone_3512P_Inline_P23.62x7.27mm_D1.02x2.41x1.02x1.57mm_Horizontal"
 			(at 66.04 30.988 90)
 			(effects
@@
 			)
 		)
-		(property "Footprint" ""
+		(property "Footprint" "Connector_PinHeader_2.54mm:PinHeader_1x02_P2.54mm_Vertical"
 			(at 175.26 76.2 0)
 			(effects
@@
 			)
 		)
-		(property "Footprint" ""
+		(property "Footprint" "Connector_PinHeader_2.54mm:PinHeader_1x02_P2.54mm_Vertical"
 			(at 178.435 43.18 90)
 			(effects

Commit message: Updated Footprint Library for custom footprints. Fixed PCB footprints, traces nalang kulang
Parts:
- U2: footprint (none) -> 1_CustomFootprints:TDS-ANALOG-SENSOR
- U4: footprint (none) -> 1_CustomFootprints:SRT_MPT1584EN_Module
Changed lines of the file:
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@@
 			)
 		)
-		(property "Footprint" ""
+		(property "Footprint" "1_CustomFootprints:TDS-ANALOG-SENSOR"
 			(at 54.61 102.87 0)
 			(effects
@@
 			)
 		)
-		(property "Footprint" ""
+		(property "Footprint" "1_CustomFootprints:SRT_MPT1584EN_Module"
 			(at 104.14 34.29 0)
 			(effects

Commit message: updated schematic and pcb
Parts:
- U3: footprint Package_SO:TSSOP-10_3x3mm_P0.5mm -> 1_CustomFootprints:ADS1115
Connections:
- net at C5.2, D1.1 (K), M1.1 (+)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: now also U6.3 (VCC)
- net at C3.2, C4.2, R4.1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: no longer U6.3 (VCC)
- net at U5.28 (31_IOB15A): now also R11.1
- net at U5.32 (70_IOT41B): no longer R11.1
- net at U5.33 (71_IOT41A): no longer R9.1
- net at U5.34 (72_IOT39B): no longer R8.1
- net at R8.2, SW1.1: now also U5.40 (79_IOT12B_1V8); no longer U5.35 (73_IOT39A)
- net at U5.36 (74_IOT38B): now also R9.1
- net at U5.39 (77_IOT37A): now also R8.1
- net at U5.42 (81_IOT11B_1V8): no longer U6.2 (SDA)
- net at U5.43 (82_IOT11A_1V8): no longer U6.1 (SCL)
- net at U5.44 (83_IOT10B_1V8): now also U6.2 (SDA)
- net at U5.45 (84_IOT10A_1V8): now also U6.1 (SCL)
Other:
- moved on the sheet: R8

Commit message: updated schematic and pcb
Changed lines of the file:
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@@
 	(wire
 		(pts
-			(xy 58.42 90.17) (xy 57.15 90.17)
+			(xy 58.42 93.98) (xy 57.15 93.98)
 		)
 		(stroke
@@
 	(wire
 		(pts
-			(xy 57.15 90.17) (xy 57.15 92.71)
-		)
-		(stroke
-			(width 0)
-			(type default)
-		)
-	)
-	(wire
-		(pts
-			(xy 58.42 95.25) (xy 58.42 90.17)
-		)
-		(stroke
+			(xy 57.15 93.98) (xy 57.15 92.71)
+		)
+		(stroke
+			(width 0)
+			(type default)
+		)
+	)
+	(wire
+		(pts
+			(xy 58.42 95.25) (xy 58.42 93.98)
+		)
+		(stroke
