File: hardware/Design-1-Draft.kicad_pcb (KiCad board)
At the start: 2 copper layers, 130 x 170 mm, 53 parts, among them J1 Barrel_Jack_Switch, M1 WP-1, M2 WP-2, Q1 IRLZ44N, Q2 IRLZ44N, Q3 PN2222A, SW1 Button, U3 ADS1115, U5 Tang_Nano_9K

Commit message: Updated PCB and Schem
Parts:
- removed R11: 10k, Resistor_THT:R_Axial_DIN0207_L6.3mm_D2.5mm_P10.16mm_Horizontal
- removed the R3 at (171.4, 106.0)
- removed REF**: CONV_BOB-12009, 1_CustomFootprints:CONV_BOB-12009
- added C22: 0.1u, Capacitor_THT:C_Disc_D5.0mm_W2.5mm_P5.00mm, F.Cu at (155.4, 100.5)
- added C23: 0.1u, Capacitor_THT:C_Disc_D5.0mm_W2.5mm_P5.00mm, F.Cu at (151.9, 80.5)
- added FB1: FerriteBead, Resistor_THT:R_Axial_DIN0207_L6.3mm_D2.5mm_P10.16mm_Horizontal, F.Cu at (153.5, 33.3)
- added U7: BOB-12009, 1_CustomFootprints:CONV_BOB-12009, F.Cu at (154.7, 91.1)
- R10, R8: value 100 -> 10k
- R3: value 4.7k -> 100
- R4: value 4.7k -> 10k
- R5: value 10k -> 1k
- R7: value 1k -> 150
- R9: value 10k -> 150
- moved SW1 168.8 mm to (197.8, 131.0), turned to -90 degrees
- moved C11 151.8 mm to (103.4, 47.5), turned to -90 degrees
- moved R7 149.6 mm to (99.0, 145.0), turned to 180 degrees
- moved U1 149.0 mm to (193.4, 90.5), turned to 180 degrees
- moved Q3 147.9 mm to (97.3, 64.1), turned to 90 degrees
- moved BZ1 144.9 mm to (96.9, 48.5), turned to 0 degrees
- moved U2 134.9 mm to (193.9, 69.5), turned to 180 degrees
- moved C4 121.0 mm to (148.5, 45.0), turned to -90 degrees
- moved U6 119.6 mm to (156.6, 73.0)
- moved R3 115.8 mm to (200.8, 138.0), turned to 180 degrees
- moved U5 112.5 mm to (149.9, 130.4), turned to 0 degrees
- moved R5 110.1 mm to (136.4, 101.5)
- moved U3 106.1 mm to (167.7, 42.4), turned to 90 degrees
- moved C3 105.7 mm to (148.5, 53.0)
- moved R4 105.1 mm to (190.8, 124.0)
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Connections:
- net Net-(D2-K) renamed /5V_PUMPS
- net Net-(F1-Pad1) renamed /+12V
- A1 pad 17: unconnected-(A1-3V3-Pad17) -> Net-(A1-3V3)
- A1 pad 30: Net-(A1-VIN) -> /5V_ICs
- BZ1 pad 1: Net-(A1-VIN) -> /5V_ICs
- C1 pad 1: Net-(A1-VIN) -> /5V_ICs
- C11 pad 1: Net-(A1-VIN) -> /5V_ICs
- C13 pad 2: Net-(A1-VIN) -> /5V_ICs
- C14 pad 1: Net-(A1-VIN) -> /5V_ICs
- C2 pad 2: Net-(U2-A0) -> /5V_ICs
- C20 pad 1: Net-(A1-VIN) -> /5V_ICs
- C21 pad 1: Net-(A1-VIN) -> /5V_ICs
- C3 pad 1: Net-(A1-VIN) -> GND
- C3 pad 2: GND -> /5V_ADC
- C4 pad 1: Net-(A1-VIN) -> GND
- C4 pad 2: GND -> /5V_ADC
- C6 pad 1: Net-(A1-VIN) -> /5V_ICs
- C7 pad 1: Net-(A1-VIN) -> /5V_ICs
- J1 pad 2: Net-(J1-Pad2) -> GND
- R10 pad 1: Net-(U5-31_IOB15A) -> GND
- R3 pad 1: Net-(A1-VIN) -> Net-(R3-Pad1)
- R3 pad 2: Net-(A1-SDA/A4) -> Net-(U5-69_IOT42A)
- R4 pad 1: Net-(A1-SCL/A5) -> Net-(U5-3V3)
- R4 pad 2: Net-(A1-VIN) -> Net-(R3-Pad1)
- R5 pad 1: Net-(U5-3V3) -> Net-(U5-77_IOT37A)
- R5 pad 2: Net-(R3-Pad1) -> Net-(Q3-B)
- R7 pad 1: Net-(U5-77_IOT37A) -> Net-(U5-74_IOT38B)
- R7 pad 2: Net-(Q3-B) -> Net-(Q1-G)
- R8 pad 1: Net-(U5-74_IOT38B) -> Net-(Q1-G)
- R8 pad 2: Net-(Q1-G) -> GND
- R9 pad 1: Net-(Q1-G) -> Net-(U5-73_IOT39A)
- R9 pad 2: GND -> Net-(Q2-G)
- U1 pad 6: Net-(A1-VIN) -> /5V_ICs
- U2 pad 1: Net-(A1-VIN) -> /5V_ICs
- U3 pad 8: Net-(A1-VIN) -> /5V_ADC
- U4 pad 3: Net-(J1-Pad2) -> GND
- U4 pad 4: Net-(J1-Pad2) -> GND
- U4 pad 5: Net-(A1-VIN) -> /5V_ICs
- U5 pad 14: Net-(U5-35_IOB29A) -> unconnected-(U5-35_IOB29A-Pad14)
- U5 pad 28: Net-(U5-31_IOB15A) -> unconnected-(U5-31_IOB15A-Pad28)
- U5 pad 31: Net-(A1-VIN) -> /5V_ICs
- U5 pad 32: unconnected-(U5-70_IOT41B-Pad32) -> Net-(U5-70_IOT41B)
- U5 pad 35: unconnected-(U5-73_IOT39A-Pad35) -> Net-(U5-73_IOT39A)
- U6 pad 3: Net-(A1-VIN) -> /5V_ICs
Routing:
- net /5V_ICs: track 0.00 -> 483.8 mm
- net Net-(U5-74_IOT38B): track 0.00 -> 85.2 mm
- net Net-(J1-Pad2): track 71.5 -> 0.00 mm
- net Net-(Q3-B): track 0.00 -> 64.8 mm
- net Net-(U5-73_IOT39A): track 0.00 -> 61.2 mm
- net Net-(A1-SCL/A5): track 0.00 -> 60.4 mm, vias 0 -> 2
- net Net-(A1-SDA/A4): track 0.00 -> 59.2 mm, vias 0 -> 2
- net Net-(A1-D7): track 0.00 -> 58.9 mm
- net Net-(A1-3V3): track 0.00 -> 53.3 mm, vias 0 -> 4
- net Net-(U3-AIN0): track 0.00 -> 44.5 mm
- net Net-(U5-70_IOT41B): track 0.00 -> 28.2 mm
- net Net-(U5-69_IOT42A): track 0.00 -> 27.8 mm
- net Net-(A1-VIN): track 26.5 -> 0.00 mm
- net Net-(U5-3V3): track 0.00 -> 22.0 mm
- net Net-(U3-AIN1): track 0.00 -> 21.9 mm
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- added copper zone on B.Cu, net GND
- added copper zone on F.Cu, net GND
Other:
- board size 130 x 170 mm -> 165 x 135 mm
